File: RPi_Zero_pHat_Template.sch (KiCad schematic (older format))
At the start: 2 parts, among them J1 RPi_GPIO, J2 RPi_GPIO

Commit message: PCB sent out for manufacture.
Parts:
- removed J1: RPi_GPIO, RPi_Hat:Samtec_HLE-120-02-XXX-DV-BE-XX-XX, symbol Connector-ML:RPi_GPIO
- added AE1: 0868AT43A0020E, footprints:0868AT43A0020E, symbol Device:Antenna_Chip
- added C1: 3P9, Capacitors_SMD:C_0603, symbol Device:C
- added C2: 0P3, Capacitors_SMD:C_0603, symbol Device:C
- added C3: 100N, Capacitors_SMD:C_0603, symbol Device:C
- added C4: 1U, Capacitors_SMD:C_0603, symbol Device:C
- added L1: 18N, Resistors_SMD:R_0402, symbol Device:L
- added U1: RFM69HCW, RF:RFM69HCW-XXXS2, symbol RF_Module:RFM69HCW
- J2: footprint RPi_Hat:Pin_Header_Straight_2x20 -> Connector_PinHeader_2.54mm:PinHeader_2x20_P2.54mm_Vertical
Connections:
- net labels added: +3V3, GND
- wire segments 0 -> 66
- no-connect marks 0 -> 5
Other:
- note removed: "Socket on bottom"
- note removed: "Surface Mount Connector"
