File: RFM69HCW-868-S2.kicad_pcb (KiCad board)
At the start: 2 copper layers, 75 x 30 mm, 16 parts, among them J2 RPi_GPIO, U1 RFM69HCW

Commit message: Added Gerber files and improved documentation
Other:
- board text removed: "Select one of these board edges depending upon the type of socket that is used."
