File: RFM69HCW-868-S2.sch (KiCad schematic (older format))
At the start: 8 parts, among them J2 RPi_GPIO, U1 RFM69HCW

Commit message: Renamed files to match project name
Improved documentation
Parts:
- AE1: MANF (none) -> JOHANSON; MANF# (none) -> 1885493; SUPPLIER (none) -> FARNELL; SUPPLIER# (none) -> 1885493
- C1: MANF (none) -> JOHANSON; MANF# (none) -> 251R14S3R9CV4T; SUPPLIER (none) -> FARNELL; SUPPLIER# (none) -> 1885381
- C2: MANF (none) -> JOHANSON; MANF# (none) -> 251R14S0R3AV4T; SUPPLIER (none) -> FARNELL; SUPPLIER# (none) -> 1885351
- C3: MANF (none) -> VISHAY; MANF# (none) -> VJ0603Y104KXACW1BC; SUPPLIER (none) -> FARNELL; SUPPLIER# (none) -> 2407338
- C4: MANF (none) -> AVX; MANF# (none) -> 0603YD105MAT2A; SUPPLIER (none) -> FARNELL; SUPPLIER# (none) -> 2332677
- J2: MANF (none) -> WURTH; MANF# (none) -> 61304021821; SUPPLIER (none) -> FARNELL; SUPPLIER# (none) -> 2827916
- L1: MANF (none) -> JOHANSON; MANF# (none) -> L-07C18NJV6T; SUPPLIER (none) -> FARNELL; SUPPLIER# (none) -> 1865775
- U1: MANF (none) -> HOPERF; MANF# (none) -> RFM69HCW-868-S2; SUPPLIER (none) -> MARITEX; SUPPLIER# (none) -> RFM69HCW-868S2
Changed lines of the file:
@@
 F 2 "Connector_PinHeader_2.54mm:PinHeader_2x20_P2.54mm_Vertical" H 6800 2800 60  0001 C CNN
 F 3 "" H 6800 2800 60  0000 C CNN
+F 4 "WURTH" H 6800 2800 50  0001 C CNN "MANF"
+F 5 "61304021821" H 6800 2800 50  0001 C CNN "MANF#"
+F 6 "FARNELL" H 6800 2800 50  0001 C CNN "SUPPLIER"
+F 7 "2827916" H 6800 2800 50  0001 C CNN "SUPPLIER#"
 	1    6800 2800
 	1    0    0    -1
@@
 F 2 "RF:RFM69HCW-XXXS2" H -50 4950 50  0001 C CNN
 F 3 "https://www.hoperf.com/data/upload/portal/20181127/5bfcb8284d838.pdf" H -50 4950 50  0001 C CNN
+F 4 "MARITEX" H 3250 3300 50  0001 C CNN "SUPPLIER"
+F 5 "RFM69HCW-868S2" H 3250 3300 50  0001 C CNN "SUPPLIER#"
+F 6 "HOPERF" H 3250 3300 50  0001 C CNN "MANF"
+F 7 "RFM69HCW-868-S2" H 3250 3300 50  0001 C CNN "MANF#"
 	1    3250 3300
 	1    0    0    -1
@@
 F 1 "0868AT43A0020E" H 4809 2937 50  0000 R CNN
 F 2 "footprints:0868AT43A0020E" H 4850 3075 50  0001 C CNN
-F 3 "~" H 4850 3075 50  0001 C CNN
+F 3 "http://www.farnell.com/datasheets/2280483.pdf?_ga=2.133129742.1044651491.1556565859-289093737.1544555023&_gac=1.18349131.1555367884.Cj0KCQjw19DlBRCSARIsAOnfRei64FcwOFGwHccevtvnCF1_gtAlQkzaoKMfBkZYkqlx40vjUC8V3ZkaAmTjEALw_wcB" H 4850 3075 50  0001 C CNN
+F 4 "FARNELL" H 4950 2900 50  0001 C CNN "SUPPLIER"
+F 5 "1885493" H 4950 2900 50  0001 C CNN "SUPPLIER#"
+F 6 "JOHANSON" H 4950 2900 50  0001 C CNN "MANF"
+F 7 "1885493" H 4950 2900 50  0001 C CNN "MANF#"
 	1    4950 2900
 	-1   0    0    -1
@@
 F 1 "3P9" H 4165 3255 50  0000 L CNN
 F 2 "Capacitors_SMD:C_0603" H 4088 3150 50  0001 C CNN
-F 3 "~" H 4050 3300 50  0001 C CNN
+F 3 "http://www.farnell.com/datasheets/1731432.pdf?_ga=2.28182204.1044651491.1556565859-289093737.1544555023&_gac=1.19854794.1555367884.Cj0KCQjw19DlBRCSARIsAOnfRei64FcwOFGwHccevtvnCF1_gtAlQkzaoKMfBkZYkqlx40vjUC8V3ZkaAmTjEALw_wcB" H 4050 3300 50  0001 C CNN
+F 4 "JOHANSON" H 4050 3300 50  0001 C CNN "MANF"
+F 5 "251R14S3R9CV4T" H 4050 3300 50  0001 C CNN "MANF#"
+F 6 "FARNELL" H 4050 3300 50  0001 C CNN "SUPPLIER"
+F 7 "1885381" H 4050 3300 50  0001 C CNN "SUPPLIER#"
 	1    4050 3300
 	1    0    0    -1
@@
 F 1 "0P3" H 4565 3255 50  0000 L CNN
 F 2 "Capacitors_SMD:C_0603" H 4488 3150 50  0001 C CNN
-F 3 "~" H 4450 3300 50  0001 C CNN
+F 3 "http://www.farnell.com/datasheets/1731432.pdf?_ga=2.99920414.1044651491.1556565859-289093737.1544555023&_gac=1.26737999.1555367884.Cj0KCQjw19DlBRCSARIsAOnfRei64FcwOFGwHccevtvnCF1_gtAlQkzaoKMfBkZYkqlx40vjUC8V3ZkaAmTjEALw_wcB" H 4450 3300 50  0001 C CNN
+F 4 "JOHANSON" H 4450 3300 50  0001 C CNN "MANF"
+F 5 "251R14S0R3AV4T" H 4450 3300 50  0001 C CNN "MANF#"
+F 6 "FARNELL" H 4450 3300 50  0001 C CNN "SUPPLIER"
+F 7 "1885351" H 4450 3300 50  0001 C CNN "SUPPLIER#"
 	1    4450 3300
 	1    0    0    -1
@@
 F 1 "18N" V 4349 3000 50  0000 C CNN
 F 2 "Resistors_SMD:R_0402" H 4250 3000 50  0001 C CNN
-F 3 "~" H 4250 3000 50  0001 C CNN
+F 3 "http://www.farnell.com/datasheets/2372621.pdf?_ga=2.99903646.1044651491.1556565859-289093737.1544555023&_gac=1.255643898.1555367884.Cj0KCQjw19DlBRCSARIsAOnfRei64FcwOFGwHccevtvnCF1_gtAlQkzaoKMfBkZYkqlx40vjUC8V3ZkaAmTjEALw_wcB" H 4250 3000 50  0001 C CNN
+F 4 "FARNELL" V 4250 3000 50  0001 C CNN "SUPPLIER"
+F 5 "1865775" V 4250 3000 50  0001 C CNN "SUPPLIER#"
+F 6 "JOHANSON" V 4250 3000 50  0001 C CNN "MANF"
+F 7 "L-07C18NJV6T" V 4250 3000 50  0001 C CNN "MANF#"
 	1    4250 3000
 	0    -1   -1   0
@@
 F 1 "100N" H 2465 2555 50  0000 L CNN
 F 2 "Capacitors_SMD:C_0603" H 2388 2450 50  0001 C CNN
-F 3 "~" H 2350 2600 50  0001 C CNN
+F 3 "http://www.farnell.com/datasheets/2244871.pdf?_ga=2.95289884.1044651491.1556565859-289093737.1544555023&_gac=1.26614863.1555367884.Cj0KCQjw19DlBRCSARIsAOnfRei64FcwOFGwHccevtvnCF1_gtAlQkzaoKMfBkZYkqlx40vjUC8V3ZkaAmTjEALw_wcB" H 2350 2600 50  0001 C CNN
+F 4 "VISHAY" H 2350 2600 50  0001 C CNN "MANF"
+F 5 "VJ0603Y104KXACW1BC" H 2350 2600 50  0001 C CNN "MANF#"
+F 6 "FARNELL" H 2350 2600 50  0001 C CNN "SUPPLIER"
+F 7 "2407338" H 2350 2600 50  0001 C CNN "SUPPLIER#"
 	1    2350 2600
 	1    0    0    -1
@@
 F 1 "1U" H 2865 2555 50  0000 L CNN
 F 2 "Capacitors_SMD:C_0603" H 2788 2450 50  0001 C CNN
-F 3 "~" H 2750 2600 50  0001 C CNN
+F 3 "http://www.farnell.com/datasheets/2237828.pdf?_ga=2.64948655.1044651491.1556565859-289093737.1544555023&_gac=1.263000574.1555367884.Cj0KCQjw19DlBRCSARIsAOnfRei64FcwOFGwHccevtvnCF1_gtAlQkzaoKMfBkZYkqlx40vjUC8V3ZkaAmTjEALw_wcB" H 2750 2600 50  0001 C CNN
+F 4 "AVX" H 2750 2600 50  0001 C CNN "MANF"
+F 5 "0603YD105MAT2A" H 2750 2600 50  0001 C CNN "MANF#"
+F 6 "FARNELL" H 2750 2600 50  0001 C CNN "SUPPLIER"
+F 7 "2332677" H 2750 2600 50  0001 C CNN "SUPPLIER#"
 	1    2750 2600
 	1    0    0    -1
